File: myMechanicalKeybaord/RGB_MATRIX.kicad_sch (KiCad schematic)
At the start: 82 parts

Commit message: Add lock files for MechanicalKeyboard schematic and PCB autosave
Parts:
- renumbered D279 to D167, D294 to D168, D175 to D169, D280 to D170, D295 to D171, D310 to D172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
