File: myMechanicalKeybaord/White_led.kicad_sch (KiCad schematic)
At the start: 82 parts

Commit message: Add lock files for MechanicalKeyboard schematic and PCB autosave
Parts:
- renumbered D99 to D100, D100 to D101, D101 to D102, D102 to D103, D103 to D104, D104 to D105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
