File: myMechanicalKeybaord/MechanicalKeyboard.kicad_sch (KiCad schematic)
At the start: 167 parts, among them P1 USB_C_Plug_USB2.0, SW1 SW_Push, SW10 SW_Push, SW11 SW_Push, SW12 SW_Push, SW13 SW_Push, SW14 SW_Push, SW15 SW_Push, SW16 SW_Push, SW17 SW_Push, SW18 SW_Push, SW19 SW_Push, SW2 SW_Push, SW20 SW_Push, SW21 SW_Push, SW22 SW_Push, SW23 SW_Push, SW24 SW_Push, SW25 SW_Push, SW26 SW_Push, SW27 SW_Push, SW28 SW_Push, SW29 SW_Push, SW3 SW_Push, SW30 SW_Push, SW31 SW_Push, SW32 SW_Push, SW33 SW_Push, SW34 SW_Push, SW35 SW_Push, SW36 SW_Push, SW37 SW_Push, SW38 SW_Push, SW39 SW_Push, SW4 SW_Push, SW40 SW_Push, SW41 SW_Push, SW42 SW_Push, SW43 SW_Push, SW44 SW_Push, SW45 SW_Push, SW46 SW_Push, SW47 SW_Push, SW48 SW_Push, SW49 SW_Push, SW5 SW_Push, SW50 SW_Push, SW51 SW_Push, SW52 SW_Push, SW53 SW_Push, SW54 SW_Push, SW55 SW_Push, SW56 SW_Push, SW57 SW_Push, SW58 SW_Push, SW59 SW_Push, SW6 SW_Push, SW60 SW_Push, SW61 SW_Push, SW62 SW_Push, SW63 SW_Push, SW64 SW_Push, SW65 SW_Push, SW66 SW_Push, SW67 SW_Push, SW68 SW_Push, SW69 SW_Push, SW7 SW_Push, SW70 SW_Push, SW71 SW_Push, SW72 SW_Push, SW73 SW_Push, SW74 SW_Push, SW75 SW_Push, SW76 SW_Push, SW77 SW_Push, SW78 SW_Push, SW79 SW_Push, SW8 SW_Push, SW80 SW_Push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

Commit message: Add lock file for MechanicalKeyboard project with hostname and username
Parts:
- removed P1: USB_C_Plug_USB2.0, symbol Connector:USB_C_Plug_USB2.0
- removed U1: nRF52840, Package_DFN_QFN:Nordic_AQFN-73-1EP_7x7mm_P0.5mm, symbol MCU_Nordic:nRF52840
- added C1, C10, C11, C12, C13, C14, C2, C3, C4, C5, C6, C7, C8, C9: C, symbol Device:C
- added D166, D84: LED, symbol Device:LED
- added J1: USB_C_Receptacle_USB2.0_16P, symbol Connector:USB_C_Receptacle_USB2.0_16P
- added L1, L2, L3: L, symbol Device:L
- added R1, R2: 5.1k, symbol Device:R
- added R3, R4, R5, R6, R7, R8, R9: R, symbol Device:R
- added SW83: SW_Push, symbol Switch:SW_Push
- added TP1, TP2: TestPoint, symbol Connector:TestPoint
- added U1: TP4056-42-ESOP8, Package_SO:SOIC-8-1EP_3.9x4.9mm_P1.27mm_EP2.41x3.3mm_ThermalVias, symbol Battery_Management:TP4056-42-ESOP8
- added U3: NRF52840-QFAA-R7, footprints:QFN48_NRF52840-QFAA-R7_NOR-L, symbol 2026-05-13_14-14-24:NRF52840-QFAA-R7
- added U4: DW01-A, SOT23-6_1P7X3P02-0P95_SFE, symbol 2026-05-14_13-39-16:DW01-A
- added U5: ~, symbol FS8205A:FS8205_A
- added U6: USBLC6-2P6, Package_TO_SOT_SMD:SOT-666, symbol Power_Protection:USBLC6-2P6
- added Y1, Y2: Crystal, symbol Device:Crystal
Connections:
- net GND: now also C10.2, C11.2, C12.1, C13.1, C14.2, C2.1, C3.1, C4.2, C5.1, C6.1, C7.2, C8.2, C9.2, J1.A1 (GND), J1.A12 (GND), J1.B1 (GND), J1.B12 (GND), J1.S1 (SHIELD), R1.2, R2.2, R4.1, R7.1, R9.2, SW83.1, U1.1 (TEMP), U1.3 (GND), U3.32 (VSS_PA), U3.45 (VSS), U3.49 (VSS), U5.6 (S2), U5.7 (S2), U6.2 (GND)
- new net: C11.1, U3.35 (XC1), Y1.1
- new net: SW83.2, U3.16
- new net: C12.2, U3.2, Y2.1
- new net: TP2.1, U3.26 (SWDIO)
- new net: TP1.1, U3.27 (SWDCLK)
- new net: C13.2, U3.3, Y2.2
- new net: L1.1, U3.31 (ANT)
- new net: C14.1, U3.33 (DEC6)
- new net: C10.1, U3.36 (XC2), Y1.2
- new net: C9.1, U3.46 (DEC4)
- new net: L3.2, U3.47 (DCC)
- new net: C3.2, L1.2, L2.1
- new net: J1.A5 (CC1), R1.1
- new net: J1.B5 (CC2), R2.1
- new net: U4.1 (DOUT), U5.4 (G1)
- new net: R7.2, U4.2 (VM)
- new net: U4.3 (COUT), U5.5 (G2)
- new net: C1.1, R3.1, U4.5 (VDD)
- new net: C1.2, U4.6 (VSS)
- new net: R4.2, U1.2 (PROG)
- new net: R5.1, U1.6 (~{STDBY})
- new net: R6.1, U1.7 (~{CHRG})
- new net: D84.1 (K), R5.2
- new net: D166.1 (K), R6.2
- new net +3.3V: C4.1, C5.2, C6.2, C7.1, C8.1, L3.1, U3.12 (VDD), U3.17 (VDD), U3.25 (VDD), U3.37 (VDD), U3.48 (VDD)
- new net +5V: J1.A4 (VBUS), J1.A9 (VBUS), J1.B4 (VBUS), J1.B9 (VBUS)
- new net ANTENNA: L2.2
- new net B+: R3.2, R8.1, U1.5 (BAT)
- new net B-: U5.2 (S1), U5.3 (S1)
- new net B_PIN: R8.2, R9.1
- new net Conn_D+: U6.6 (I/O1)
- new net Conn_D-: U6.4 (I/O2)
- new net D+: J1.A6 (D+), J1.B6 (D+), U6.1 (I/O1)
- new net D-: J1.A7 (D-), J1.B7 (D-), U6.3 (I/O2)
- new net VBUS: C2.2, D166.2 (A), D84.2 (A), U1.4 (V_{CC}), U1.8 (CE), U6.5 (VBUS)
- no-connect marks 0 -> 3
Other:
- moved on the sheet: U2

Commit message: Add lock files for MechanicalKeyboard schematic and PCB autosave
Parts:
- removed C14: C, symbol Device:C
- added C3, C6, C9: C, Capacitor_SMD:C_0603_1608Metric, symbol Device:C
- added TP1, TP2, TP4: TestPoint, TestPoint:TestPoint_Pad_D1.0mm, symbol Connector:TestPoint
- C1: renamed from C12; footprint (none) -> Capacitor_SMD:CP_Elec_3x5.3
- C10: renamed from C8; footprint (none) -> Capacitor_SMD:C_0603_1608Metric
- C11: renamed from C7; footprint (none) -> Capacitor_SMD:C_0603_1608Metric
- C12: renamed from C3; footprint (none) -> Capacitor_SMD:C_0603_1608Metric
- C13: renamed from C10; footprint (none) -> Capacitor_SMD:C_0603_1608Metric
- C14: renamed from C11; footprint (none) -> Capacitor_SMD:C_0603_1608Metric
- C15: renamed from C2; footprint (none) -> Capacitor_SMD:C_0603_1608Metric
- C16: renamed from C1; footprint (none) -> Capacitor_SMD:C_0603_1608Metric
- C2: renamed from C13; footprint (none) -> Capacitor_SMD:C_0603_1608Metric
- C4: renamed from C5; footprint (none) -> Capacitor_SMD:C_0603_1608Metric
- C5: renamed from C6; footprint (none) -> Capacitor_SMD:C_0603_1608Metric
- C7: renamed from C4; footprint (none) -> Capacitor_SMD:C_0603_1608Metric
- C8: renamed from C9; footprint (none) -> Capacitor_SMD:C_0603_1608Metric
- D35: renamed from D84; footprint (none) -> Diode_SMD:D_SOD-123
- D36: renamed from D166; footprint (none) -> Diode_SMD:D_SOD-123
- D83: renamed from D72; footprint Diode_SMD:D_SOD-123 -> LED_SMD:LED_0603_1608Metric
- D84: renamed from D82; footprint Diode_SMD:D_SOD-123 -> LED_SMD:LED_0603_1608Metric
- J1: footprint (none) -> Connector_USB:USB_C_Receptacle_HRO_TYPE-C-31-M-12
- L1, L2, L3: footprint (none) -> Inductor_SMD:L_0603_1608Metric
- R1, R2, R8, R9: footprint (none) -> Resistor_SMD:R_0201_0603Metric
- R3: renamed from R5; footprint (none) -> Resistor_SMD:R_0201_0603Metric
- R4: renamed from R6; footprint (none) -> Resistor_SMD:R_0201_0603Metric
- R5: renamed from R4; footprint (none) -> Resistor_SMD:R_0201_0603Metric
- R6: renamed from R7; footprint (none) -> Resistor_SMD:R_0201_0603Metric
- R7: renamed from R3; footprint (none) -> Resistor_SMD:R_0201_0603Metric
- SW1: renamed from SW83; footprint (none) -> Button_Switch_SMD:SW_SPST_TL3342
- TP3: renamed from TP1; footprint (none) -> TestPoint:TestPoint_Pad_D1.0mm
- TP5: renamed from TP2; footprint (none) -> TestPoint:TestPoint_Pad_D1.0mm
- U2: renamed from U1; footprint Package_SO:SOIC-8-1EP_3.9x4.9mm_P1.27mm_EP2.41x3.3mm_ThermalVias -> Package_DFN_QFN:QFN-28-1EP_4x4mm_P0.4mm_EP2.3x2.3mm
- U3: renamed from U4; footprint SOT23-6_1P7X3P02-0P95_SFE -> footprints:QFN48_NRF52840-QFAA-R7_NOR-L
- U4: renamed from U2; footprint Package_DFN_QFN:QFN-28-1EP_4x4mm_P0.4mm_EP2.3x2.3mm -> SOT23-6_1P7X3P02-0P95_SFE
- U5: footprint (none) -> FS8205A:SOP65P640X120-8N
- Y1: renamed from Y2; footprint (none) -> Crystal:Crystal_SMD_3215-2Pin_3.2x1.5mm
- Y2: renamed from Y1; footprint (none) -> Crystal:Crystal_SMD_3225-4Pin_3.2x2.5mm
- renumbered D15 to D1, D32 to D10, D46 to D11, D60 to D12, D3 to D13, D18 to D14, D33 to D15, D47 to D16, D61 to D17, D4 to D18, D30 to D2, D34 to D20, D48 to D21, D62 to D22, D5 to D23, D20 to D24, D35 to D25, D49 to D26, D63 to D27, D73 to D28, D6 to D29, D1 to D3, D21 to D30, D36 to D31, D50 to D32, D64 to D33, D74 to D34, D7 to D37, D22 to D38, D37 to D39, D16 to D4, D51 to D40, D65 to D41, D75 to D42, D8 to D43, D23 to D44, D38 to D45, D52 to D46, D66 to D47, D76 to D48, D9 to D49, D31 to D5, D24 to D50, D39 to D51, D53 to D52, D67 to D53, D77 to D54, D10 to D55, D25 to D56, D40 to D57, D54 to D58, D68 to D59, D45 to D6, D78 to D60, D11 to D61, D26 to D62, D41 to D63, D55 to D64, D69 to D65, D79 to D66, D12 to D67, D27 to D68, D42 to D69, D59 to D7, D56 to D70, D70 to D71, D80 to D72, D13 to D73, D28 to D74, D43 to D75, D57 to D76, D71 to D77, D81 to D78, D14 to D79, D2 to D8, D29 to D80, D44 to D81, D58 to D82, D17 to D9, SW17 to SW10, SW32 to SW11, SW46 to SW12, SW60 to SW13, SW3 to SW14, SW18 to SW15, SW33 to SW16, SW47 to SW17, SW61 to SW18, SW4 to SW19, SW15 to SW2, SW19 to SW20, SW34 to SW21, SW48 to SW22, SW62 to SW23, SW5 to SW24, SW20 to SW25, SW35 to SW26, SW49 to SW27, SW63 to SW28, SW73 to SW29, SW30 to SW3, SW6 to SW30, SW21 to SW31, SW36 to SW32, SW50 to SW33, SW64 to SW34, SW74 to SW35, SW7 to SW36, SW22 to SW37, SW37 to SW38, SW51 to SW39, SW1 to SW4, SW65 to SW40, SW75 to SW41, SW8 to SW42, SW23 to SW43, SW38 to SW44, SW52 to SW45, SW66 to SW46, SW76 to SW47, SW9 to SW48, SW24 to SW49, SW16 to SW5, SW39 to SW50, SW53 to SW51, SW67 to SW52, SW77 to SW53, SW10 to SW54, SW25 to SW55, SW40 to SW56, SW54 to SW57, SW68 to SW58, SW78 to SW59, SW31 to SW6, SW11 to SW60, SW26 to SW61, SW41 to SW62, SW55 to SW63, SW69 to SW64, SW79 to SW65, SW12 to SW66, SW27 to SW67, SW42 to SW68, SW56 to SW69, SW45 to SW7, SW80 to SW71, SW13 to SW72, SW28 to SW73, SW43 to SW74, SW57 to SW75, SW71 to SW76, SW81 to SW77, SW14 to SW78, SW29 to SW79, SW59 to SW8, SW44 to SW80, SW58 to SW81, SW72 to SW82, SW82 to SW83, SW2 to SW9, U3 to U1
Connections:
- net +3.3V: now also C6.1, TP2.1
- net GND: now also C3.2, C6.2, C9.2, TP4.1
- net at U1.1 (DEC1): now also C3.1
- net at SW1.2, U1.16: now also TP1.1
- net at U1.33 (DEC6): now also C8.1, U1.46 (DEC4)
- net at U1.34 (DEC3): now also C9.1

Commit message: Update KiCad project files and make various improvements
- Modified visible layers in MechanicalKeyboard.kicad_prl for better visibility.
- Increased minimum clearance in MechanicalKeyboard.kicad_pro from 0.0 to 0.5 for improved design rules.
- Removed unused global labels and updated footprints in MechanicalKeyboard.kicad_sch for better component management.
- Updated footprint references for components in the schematic.
- Added new entries to fp-info-cache for DW01A footprint.
- Created an autosave file for MechanicalKeyboard.kicad_sch.
- Added multiple backup zip files for MechanicalKeyboard project.
- Created a lock file for MechanicalKeyboard.kicad_sch to prevent concurrent edits.
Parts:
- C1: footprint Capacitor_SMD:CP_Elec_3x5.3 -> Capacitor_SMD:C_0603_1608Metric
- U3: footprint footprints:QFN48_NRF52840-QFAA-R7_NOR-L -> DW01A:SOT23-6_1P7X3P02-0P95_SFE-L
- U4: footprint SOT23-6_1P7X3P02-0P95_SFE -> DW01A:SOT23-6_1P7X3P02-0P95_SFE
Connections:
- net GND: no longer C12.1
- new net VSS_PA: C12.1
Changed lines of the file:
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@@
 		)
 	)
-	(global_label "VSS_PA"
-		(shape input)
-		(at 140.97 508 270)
-		(fields_autoplaced yes)
-		(effects
-			(font
-				(size 1.27 1.27)
-			)
-			(justify right)
-		)
-		(property "Intersheetrefs" "${INTERSHEET_REFS}"
-			(at 140.97 517.819 90)
-			(effects
-				(font
-					(size 1.27 1.27)
-				)
-				(justify right)
-				(hide yes)
-			)
-		)
-	)
 	(global_label "VBAT"
 		(shape input)
@@
 			)
 		)
-		(property "Footprint" "Capacitor_SMD:CP_Elec_3x5.3"
+		(property "Footprint" "Capacitor_SMD:C_0603_1608Metric"
 			(at 54.61 444.8048 0)
 			(effects
@@
 			)
 		)
-		(property "Footprint" "footprints:QFN48_NRF52840-QFAA-R7_NOR-L"
+		(property "Footprint" "DW01A:SOT23-6_1P7X3P02-0P95_SFE-L"
 			(at 250.19 337.82 0)
 			(effects
@@
 	)
 	(symbol
-		(lib_id "power:GND")
-		(at 140.97 508 180)
-		(unit 1)
-		(exclude_from_sim no)
-		(in_bom yes)
-		(on_board yes)
-		(dnp no)
-		(fields_autoplaced yes)
-		(property "Reference" "#PWR024"
-			(at 140.97 501.65 0)
-			(effects
-				(font
-					(size 1.27 1.27)
-				)
-				(hide yes)
-			)
-		)
-		(property "Value" "GND"
-			(at 140.97 502.92 0)
-			(effects
-				(font
-					(size 1.27 1.27)
-				)
-			)
-		)
-		(property "Footprint" ""
-			(at 140.97 508 0)
-			(effects
-				(font
-					(size 1.27 1.27)
-				)
-				(hide yes)
-			)
-		)
-		(property "Datasheet" ""
-			(at 140.97 508 0)
-			(effects
-				(font
-					(size 1.27 1.27)
-				)
-				(hide yes)
-			)
-		)
-		(property "Description" "Power symbol creates a global label with name \"GND\" , ground"
-			(at 140.97 508 0)
-			(effects
-				(font
-					(size 1.27 1.27)
-				)
-				(hide yes)
-			)
-		)
-		(pin "1"
-		)
-		(instances
-			(project "MechanicalKeyboard"
-				(path "/dd8f9092-0812-4ba5-9c06-768857751bc0"
-					(reference "#PWR024")
-					(unit 1)
-				)
-			)
-		)
-	)
-	(symbol
 		(lib_id "Device:C")
 		(at 50.8 453.39 90)
@@
 			)
 		)
-		(property "Footprint" "SOT23-6_1P7X3P02-0P95_SFE"
+		(property "Footprint" "DW01A:SOT23-6_1P7X3P02-0P95_SFE"
 			(at 260.35 497.84 0)
 			(effects

Commit message: Update mechanical keyboard project files with various enhancements and new components
- Changed high contrast mode setting in MechanicalKeyboard.kicad_prl for improved visibility.
- Adjusted net color opacity settings for better clarity in MechanicalKeyboard.kicad_prl.
- Modified via diameter in MechanicalKeyboard.kicad_pro for optimized routing.
- Added new global label "VBUS" in MechanicalKeyboard.kicad_sch for power distribution.
- Removed duplicate "VBUS" global label to streamline schematic.
- Updated footprint references in MechanicalKeyboard.kicad_sch for the TP4056 component.
- Added new footprint entries for TP4056 in fp-info-cache for better component management.
- Created multiple backup zip files for MechanicalKeyboard project to ensure data safety.
Parts:
- U2: footprint Package_DFN_QFN:QFN-28-1EP_4x4mm_P0.4mm_EP2.3x2.3mm -> TP_4056_ESOP8:TP4056-42-ESOP8_TPW
Changed lines of the file:
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@@
 		)
 	)
+	(global_label "VBUS"
+		(shape input)
+		(at 226.06 330.2 90)
+		(fields_autoplaced yes)
+		(effects
+			(font
+				(size 1.27 1.27)
+			)
+			(justify left)
+		)
+		(property "Intersheetrefs" "${INTERSHEET_REFS}"
+			(at 226.06 322.3162 90)
+			(effects
+				(font
+					(size 1.27 1.27)
+				)
+				(justify left)
+				(hide yes)
+			)
+		)
+	)
 	(global_label "COL 14"
 		(shape input)
@@
 		)
 	)
-	(global_label "VBUS"
-		(shape input)
-		(at 226.06 330.2 90)
-		(fields_autoplaced yes)
-		(effects
-			(font
-				(size 1.27 1.27)
-			)
-			(justify left)
-		)
-		(property "Intersheetrefs" "${INTERSHEET_REFS}"
-			(at 226.06 322.3162 90)
-			(effects
-				(font
-					(size 1.27 1.27)
-				)
-				(justify left)
-				(hide yes)
-			)
-		)
-	)
 	(global_label "COL 13"
 		(shape input)
@@
 			)
 		)
-		(property "Footprint" "Package_DFN_QFN:QFN-28-1EP_4x4mm_P0.4mm_EP2.3x2.3mm"
+		(property "Footprint" "TP_4056_ESOP8:TP4056-42-ESOP8_TPW"
 			(at 226.568 365.76 0)
 			(effects
@@
 					(size 1.27 1.27)
 				)
-				(hide yes)
 			)
 		)

Commit message: Update active layer and add test point in schematic
- Changed the active layer from 0 to 2 in MechanicalKeyboard.kicad_prl.
- Added a new junction and wire connections at coordinates (140.97, 490.22) in MechanicalKeyboard.kicad_sch.
- Introduced a test point symbol (TP6) with associated properties and connections in the schematic.
- Updated footprint properties for several components, swapping between LED and Diode footprints as necessary.
- Added multiple backup files for the MechanicalKeyboard project.
Parts:
- added TP6: TestPoint, TestPoint:TestPoint_Pad_D1.0mm, symbol Connector:TestPoint
- D35, D36: footprint Diode_SMD:D_SOD-123 -> LED_SMD:LED_0603_1608Metric
- D83, D84: footprint LED_SMD:LED_0603_1608Metric -> Diode_SMD:D_SOD-123
Connections:
- net ANTENNA: now also TP6.1
Changed lines of the file:
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@@
 	)
 	(junction
+		(at 140.97 490.22)
+		(diameter 0)
+		(color 0 0 0 0)
+	)
+	(junction
 		(at 311.15 345.44)
 		(diameter 0)
@@
 	(wire
 		(pts
-			(xy 139.7 490.22) (xy 142.24 490.22)
+			(xy 139.7 490.22) (xy 140.97 490.22)
 		)
 		(stroke
@@
 	(wire
 		(pts
+			(xy 140.97 490.22) (xy 142.24 490.22)
+		)
+		(stroke
+			(width 0)
+			(type default)
+		)
+	)
+	(wire
+		(pts
 			(xy 248.92 351.79) (xy 248.92 337.82)
 		)
@@
 	)
 	(symbol
+		(lib_id "Connector:TestPoint")
+		(at 140.97 490.22 180)
+		(unit 1)
+		(exclude_from_sim no)
+		(in_bom yes)
+		(on_board yes)
+		(dnp no)
+		(property "Reference" "TP6"
+			(at 142.24 492.252 90)
+			(effects
+				(font
+					(size 1.27 1.27)
+				)
+				(justify left)
+			)
+		)
+		(property "Value" "TestPoint"
+			(at 140.97 492.252 90)
+			(effects
+				(font
+					(size 1.27 1.27)
+				)
+				(justify left)
+				(hide yes)
+			)
+		)
+		(property "Footprint" "TestPoint:TestPoint_Pad_D1.0mm"
+			(at 135.89 490.22 0)
+			(effects
+				(font
+					(size 1.27 1.27)
+				)
+				(hide yes)
+			)
+		)
+		(property "Datasheet" "~"
+			(at 135.89 490.22 0)
+			(effects
+				(font
+					(size 1.27 1.27)
+				)
+				(hide yes)
+			)
+		)
+		(property "Description" "test point"
+			(at 140.97 490.22 0)
+			(effects
+				(font
+					(size 1.27 1.27)
+				)
+				(hide yes)
+			)
+		)
+		(pin "1"
+		)
+		(instances
+			(project "MechanicalKeyboard"
+				(path "/dd8f9092-0812-4ba5-9c06-768857751bc0"
+					(reference "TP6")
+					(unit 1)
+				)
+			)
+		)
+	)
+	(symbol
 		(lib_id "Device:C")
 		(at 50.8 453.39 90)
@@
 			)
 		)
-		(property "Footprint" "LED_SMD:LED_0603_1608Metric"
+		(property "Footprint" "Diode_SMD:D_SOD-123"
 			(at 368.3 198.12 0)
 			(effects
@@
 			)
 		)
-		(property "Footprint" "LED_SMD:LED_0603_1608Metric"
+		(property "Footprint" "Diode_SMD:D_SOD-123"
 			(at 368.3 220.98 0)
 			(effects
@@
 			)
 		)
-		(property "Footprint" "Diode_SMD:D_SOD-123"
+		(property "Footprint" "LED_SMD:LED_0603_1608Metric"
 			(at 210.82 341.63 0)
 			(effects
@@
 			)
 		)
-		(property "Footprint" "Diode_SMD:D_SOD-123"
+		(property "Footprint" "LED_SMD:LED_0603_1608Metric"
 			(at 207.01 341.63 0)
 			(effects
